File: first-project/second-project/second-project.kicad_sch (KiCad schematic)
At the start: 0 parts

Commit message: second iteration
Parts:
- added BT1: Battery_Cell, Battery:BatteryHolder_Keystone_3034_1x20mm, symbol Device:Battery_Cell
- added D1, D2, D3, D4: LED, LED_THT:LED_D5.0mm, symbol Device:LED
- added R1, R2, R3, R4: R, Resistor_THT:R_Axial_DIN0207_L6.3mm_D2.5mm_P7.62mm_Horizontal, symbol Device:R
- added SW1: SW_Push, Button_Switch_THT:SW_PUSH_6mm, symbol Switch:SW_Push
Connections:
- new net: D3.2 (A), R3.1
- new net: BT1.1 (+), R1.2, R2.2, R3.2, R4.2
- new net: D1.2 (A), R1.1
- new net: D2.2 (A), R2.1
- new net: D4.2 (A), R4.1
- new net: BT1.2 (-), SW1.1
- new net: D1.1 (K), D2.1 (K), D3.1 (K), D4.1 (K), SW1.2
